Commit message: Update moveit configs for Jazzy

File: panda_moveit_config/config/panda_arm_hand.srdf.xacro (robot description, xacro)
@@ -19,10 +19,10 @@
   </group>
   <group_state name="open" group="hand">
-    <joint name="panda_finger_joint1" value="0.035" />
-    <joint name="panda_finger_joint2" value="0.035" />
+    <joint name="panda_finger_joint1" value="0.04" />
+    <joint name="panda_finger_joint2" value="0.04" />
   </group_state>
   <group_state name="close" group="hand">
-    <joint name="panda_finger_joint1" value="0.028" />
-    <joint name="panda_finger_joint2" value="0.028" />
+    <joint name="panda_finger_joint1" value="0.0" />
+    <joint name="panda_finger_joint2" value="0.0" />
   </group_state>
   <!--END EFFECTOR: Purpose: Represent information about an end effector.-->

File: panda_moveit_config/config/panda_hand.ros2_control.xacro (robot description, xacro)
@@ -25,5 +25,4 @@
                 <param name="mimic">panda_finger_joint1</param>
                 <param name="multiplier">1</param>
-                <command_interface name="position" />
                 <state_interface name="position">
                   <param name="initial_value">0.0</param>
